Commit message: feat: add standalone pick and place demo

File: ros_ws/src/test/standalone_manipulation_test/urdf/stoneware_arm.urdf.xacro (robot description, xacro)
@@ -6,6 +6,6 @@
   <xacro:property name="base_height" value="0.70"/>
   <xacro:property name="rail_height" value="0.10"/>
-  <xacro:property name="radial_offset" value="0.30"/>
-  <xacro:property name="tool_offset" value="0.12"/>
+  <xacro:property name="radial_offset" value="0.65"/>
+  <xacro:property name="tool_offset" value="0.305"/>
   <material name="base_gray">
     <color rgba="0.35 0.38 0.42 1"/>
@@ -160,5 +160,5 @@
     <origin xyz="${radial_offset} 0 0" rpy="0 0 0"/>
     <axis xyz="1 0 0"/>
-    <limit lower="0.0" upper="0.70" effort="150" velocity="0.40"/>
+    <limit lower="-0.35" upper="0.35" effort="150" velocity="0.40"/>
   </joint>
   <joint name="lift_joint" type="prismatic">
@@ -167,5 +167,5 @@
     <origin xyz="0 0 0" rpy="0 0 0"/>
     <axis xyz="0 0 1"/>
-    <limit lower="-0.35" upper="0.25" effort="120" velocity="0.25"/>
+    <limit lower="-0.165" upper="0.435" effort="120" velocity="0.25"/>
   </joint>
   <joint name="tool_fixed_joint" type="fixed">
@@ -196,8 +196,25 @@
   <gazebo>
     <plugin
+      filename="gz-sim-pose-publisher-system"
+      name="gz::sim::systems::PosePublisher">
+      <publish_link_pose>true</publish_link_pose>
+      <publish_nested_model_pose>false</publish_nested_model_pose>
+      <use_pose_vector_msg>true</use_pose_vector_msg>
+    </plugin>
+    <plugin
       filename="libgz_ros2_control-system.so"
       name="gz_ros2_control::GazeboSimROS2ControlPlugin">
       <parameters>$(arg controllers_file)</parameters>
     </plugin>
+    <plugin
+      filename="gz-sim-detachable-joint-system"
+      name="gz::sim::systems::DetachableJoint">
+      <parent_link>lift_link</parent_link>
+      <child_model>workpiece</child_model>
+      <child_link>cylinder_link</child_link>
+      <detach_topic>/workpiece/detach</detach_topic>
+      <attach_topic>/workpiece/attach</attach_topic>
+      <output_topic>/workpiece/state</output_topic>
+    </plugin>
   </gazebo>
 </robot>
