Commit message: feat: add three-axis manipulation arm
Co-authored-by: Copilot <223556219+Copilot@users.noreply.github.com>

File: ros_ws/src/test/standalone_manipulation_test/urdf/stoneware_arm.urdf.xacro (robot description, xacro)
@@ -1,21 +1,22 @@
 <?xml version="1.0"?>
-<robot xmlns:xacro="http://www.ros.org/wiki/xacro" name="stoneware_arm">
+<robot xmlns:xacro="http://www.ros.org/wiki/xacro" name="stoneware_manipulator">
   <xacro:arg
     name="controllers_file"
     default="$(find stoneware_manipulation_test)/config/controllers.yaml"/>
-  <xacro:property name="base_radius" value="0.12"/>
-  <xacro:property name="base_height" value="0.25"/>
-  <xacro:property name="upper_arm_length" value="0.50"/>
-  <xacro:property name="upper_arm_radius" value="0.045"/>
-  <xacro:property name="forearm_length" value="0.40"/>
-  <xacro:property name="forearm_radius" value="0.035"/>
+  <xacro:property name="base_height" value="0.70"/>
+  <xacro:property name="rail_height" value="0.10"/>
+  <xacro:property name="radial_offset" value="0.30"/>
+  <xacro:property name="tool_offset" value="0.12"/>
   <material name="base_gray">
     <color rgba="0.35 0.38 0.42 1"/>
   </material>
-  <material name="upper_arm_blue">
+  <material name="rail_blue">
     <color rgba="0.15 0.35 0.75 1"/>
   </material>
-  <material name="forearm_orange">
+  <material name="carriage_orange">
     <color rgba="0.85 0.42 0.12 1"/>
+  </material>
+  <material name="tool_black">
+    <color rgba="0.12 0.12 0.14 1"/>
   </material>
   <link name="world"/>
@@ -23,17 +24,17 @@
     <inertial>
       <origin xyz="0 0 ${base_height / 2}" rpy="0 0 0"/>
-      <mass value="5.0"/>
+      <mass value="12.0"/>
       <inertia
-        ixx="${5.0 * (3 * base_radius ** 2 + base_height ** 2) / 12}"
+        ixx="${12.0 * (3 * 0.16 ** 2 + base_height ** 2) / 12}"
         ixy="0"
         ixz="0"
-        iyy="${5.0 * (3 * base_radius ** 2 + base_height ** 2) / 12}"
+        iyy="${12.0 * (3 * 0.16 ** 2 + base_height ** 2) / 12}"
         iyz="0"
-        izz="${5.0 * base_radius ** 2 / 2}"/>
+        izz="${12.0 * 0.16 ** 2 / 2}"/>
     </inertial>
     <visual>
       <origin xyz="0 0 ${base_height / 2}" rpy="0 0 0"/>
       <geometry>
-        <cylinder radius="${base_radius}" length="${base_height}"/>
+        <cylinder radius="0.16" length="${base_height}"/>
       </geometry>
       <material name="base_gray"/>
@@ -42,57 +43,96 @@
       <origin xyz="0 0 ${base_height / 2}" rpy="0 0 0"/>
       <geometry>
-        <cylinder radius="${base_radius}" length="${base_height}"/>
-      </geometry>
-    </collision>
-  </link>
-  <link name="upper_arm_link">
-    <inertial>
-      <origin xyz="${upper_arm_length / 2} 0 0" rpy="0 0 0"/>
-      <mass value="2.0"/>
+        <cylinder radius="0.16" length="${base_height}"/>
+      </geometry>
+    </collision>
+  </link>
+  <link name="turntable_link">
+    <inertial>
+      <origin xyz="0 0 0.04" rpy="0 0 0"/>
+      <mass value="3.0"/>
+      <inertia ixx="0.0324" ixy="0" ixz="0" iyy="0.0324" iyz="0" izz="0.0600"/>
+    </inertial>
+    <visual>
+      <origin xyz="0 0 0.04" rpy="0 0 0"/>
+      <geometry>
+        <cylinder radius="0.20" length="0.08"/>
+      </geometry>
+      <material name="base_gray"/>
+    </visual>
+    <collision>
+      <origin xyz="0 0 0.04" rpy="0 0 0"/>
+      <geometry>
+        <cylinder radius="0.20" length="0.08"/>
+      </geometry>
+    </collision>
+  </link>
+  <link name="rail_link">
+    <inertial>
+      <origin xyz="0.55 0 0" rpy="0 0 0"/>
+      <mass value="1.5"/>
       <inertia
-        ixx="${2.0 * upper_arm_radius ** 2 / 2}"
+        ixx="0.001225"
         ixy="0"
         ixz="0"
-        iyy="${2.0 * (3 * upper_arm_radius ** 2 + upper_arm_length ** 2) / 12}"
+        iyy="0.1518625"
         iyz="0"
-        izz="${2.0 * (3 * upper_arm_radius ** 2 + upper_arm_length ** 2) / 12}"/>
-    </inertial>
-    <visual>
-      <origin xyz="${upper_arm_length / 2} 0 0" rpy="0 ${pi / 2} 0"/>
-      <geometry>
-        <cylinder radius="${upper_arm_radius}" length="${upper_arm_length}"/>
-      </geometry>
-      <material name="upper_arm_blue"/>
-    </visual>
-    <collision>
-      <origin xyz="${upper_arm_length / 2} 0 0" rpy="0 ${pi / 2} 0"/>
-      <geometry>
-        <cylinder radius="${upper_arm_radius}" length="${upper_arm_length}"/>
-      </geometry>
-    </collision>
-  </link>
-  <link name="forearm_link">
-    <inertial>
-      <origin xyz="${forearm_length / 2} 0 0" rpy="0 0 0"/>
-      <mass value="1.2"/>
-      <inertia
-        ixx="${1.2 * forearm_radius ** 2 / 2}"
-        ixy="0"
-        ixz="0"
-        iyy="${1.2 * (3 * forearm_radius ** 2 + forearm_length ** 2) / 12}"
-        iyz="0"
-        izz="${1.2 * (3 * forearm_radius ** 2 + forearm_length ** 2) / 12}"/>
-    </inertial>
-    <visual>
-      <origin xyz="${forearm_length / 2} 0 0" rpy="0 ${pi / 2} 0"/>
-      <geometry>
-        <cylinder radius="${forearm_radius}" length="${forearm_length}"/>
-      </geometry>
-      <material name="forearm_orange"/>
-    </visual>
-    <collision>
-      <origin xyz="${forearm_length / 2} 0 0" rpy="0 ${pi / 2} 0"/>
-      <geometry>
-        <cylinder radius="${forearm_radius}" length="${forearm_length}"/>
+        izz="0.1518625"/>
+    </inertial>
+    <visual>
+      <origin xyz="0.55 0 0" rpy="0 0 0"/>
+      <geometry>
+        <box size="1.10 0.07 0.07"/>
+      </geometry>
+      <material name="rail_blue"/>
+    </visual>
+  </link>
+  <link name="radial_carriage_link">
+    <inertial>
+      <mass value="1.0"/>
+      <inertia ixx="0.003333" ixy="0" ixz="0" iyy="0.003033" iyz="0" izz="0.003667"/>
+    </inertial>
+    <visual>
+      <geometry>
+        <box size="0.14 0.16 0.12"/>
+      </geometry>
+      <material name="carriage_orange"/>
+    </visual>
+    <collision>
+      <geometry>
+        <box size="0.14 0.16 0.12"/>
+      </geometry>
+    </collision>
+  </link>
+  <link name="lift_link">
+    <inertial>
+      <mass value="0.8"/>
+      <inertia ixx="0.002133" ixy="0" ixz="0" iyy="0.002133" iyz="0" izz="0.000683"/>
+    </inertial>
+    <visual>
+      <geometry>
+        <box size="0.08 0.08 0.16"/>
+      </geometry>
+      <material name="base_gray"/>
+    </visual>
+    <collision>
+      <geometry>
+        <box size="0.08 0.08 0.16"/>
+      </geometry>
+    </collision>
+  </link>
+  <link name="tool_link">
+    <inertial>
+      <mass value="0.25"/>
+      <inertia ixx="0.000209" ixy="0" ixz="0" iyy="0.000209" iyz="0" izz="0.000378"/>
+    </inertial>
+    <visual>
+      <geometry>
+        <cylinder radius="0.055" length="0.03"/>
+      </geometry>
+      <material name="tool_black"/>
+    </visual>
+    <collision>
+      <geometry>
+        <cylinder radius="0.055" length="0.03"/>
       </geometry>
     </collision>
@@ -103,17 +143,34 @@
     <origin xyz="0 0 0" rpy="0 0 0"/>
   </joint>
-  <joint name="shoulder_joint" type="revolute">
+  <joint name="yaw_joint" type="revolute">
     <parent link="base_link"/>
-    <child link="upper_arm_link"/>
+    <child link="turntable_link"/>
     <origin xyz="0 0 ${base_height}" rpy="0 0 0"/>
-    <axis xyz="0 1 0"/>
-    <limit lower="-1.57" upper="1.57" effort="50" velocity="1.5"/>
-  </joint>
-  <joint name="elbow_joint" type="revolute">
-    <parent link="upper_arm_link"/>
-    <child link="forearm_link"/>
-    <origin xyz="${upper_arm_length} 0 0" rpy="0 0 0"/>
-    <axis xyz="0 1 0"/>
-    <limit lower="-2.35" upper="2.35" effort="30" velocity="2.0"/>
+    <axis xyz="0 0 1"/>
+    <limit lower="-3.14159" upper="3.14159" effort="30" velocity="1.2"/>
+  </joint>
+  <joint name="rail_fixed_joint" type="fixed">
+    <parent link="turntable_link"/>
+    <child link="rail_link"/>
+    <origin xyz="0 0 ${rail_height}" rpy="0 0 0"/>
+  </joint>
+  <joint name="radial_joint" type="prismatic">
+    <parent link="rail_link"/>
+    <child link="radial_carriage_link"/>
+    <origin xyz="${radial_offset} 0 0" rpy="0 0 0"/>
+    <axis xyz="1 0 0"/>
+    <limit lower="0.0" upper="0.70" effort="150" velocity="0.40"/>
+  </joint>
+  <joint name="lift_joint" type="prismatic">
+    <parent link="radial_carriage_link"/>
+    <child link="lift_link"/>
+    <origin xyz="0 0 0" rpy="0 0 0"/>
+    <axis xyz="0 0 1"/>
+    <limit lower="-0.35" upper="0.25" effort="120" velocity="0.25"/>
+  </joint>
+  <joint name="tool_fixed_joint" type="fixed">
+    <parent link="lift_link"/>
+    <child link="tool_link"/>
+    <origin xyz="0 0 -${tool_offset}" rpy="0 0 0"/>
   </joint>
   <ros2_control name="GazeboSimSystem" type="system">
@@ -121,10 +178,15 @@
       <plugin>gz_ros2_control/GazeboSimSystem</plugin>
     </hardware>
-    <joint name="shoulder_joint">
+    <joint name="yaw_joint">
       <command_interface name="position"/>
       <state_interface name="position"/>
       <state_interface name="velocity"/>
     </joint>
-    <joint name="elbow_joint">
+    <joint name="radial_joint">
+      <command_interface name="position"/>
+      <state_interface name="position"/>
+      <state_interface name="velocity"/>
+    </joint>
+    <joint name="lift_joint">
       <command_interface name="position"/>
       <state_interface name="position"/>

Commit message: feat: improve standalone demo presentation
Add headless launch argument forwarding and refine the robot and world visuals.

Co-authored-by: Copilot <223556219+Copilot@users.noreply.github.com>

File: ros_ws/src/test/standalone_manipulation_test/urdf/stoneware_arm.urdf.xacro (robot description, xacro)
@@ -9,14 +9,20 @@
   <xacro:property name="tool_offset" value="0.305"/>
   <material name="base_gray">
-    <color rgba="0.35 0.38 0.42 1"/>
+    <color rgba="0.16 0.20 0.24 1"/>
   </material>
   <material name="rail_blue">
-    <color rgba="0.15 0.35 0.75 1"/>
+    <color rgba="0.12 0.31 0.43 1"/>
   </material>
   <material name="carriage_orange">
-    <color rgba="0.85 0.42 0.12 1"/>
+    <color rgba="0.94 0.34 0.07 1"/>
   </material>
   <material name="tool_black">
-    <color rgba="0.12 0.12 0.14 1"/>
+    <color rgba="0.08 0.10 0.12 1"/>
+  </material>
+  <material name="machined_steel">
+    <color rgba="0.60 0.68 0.70 1"/>
+  </material>
+  <material name="safety_yellow">
+    <color rgba="0.96 0.66 0.08 1"/>
   </material>
   <link name="world"/>
@@ -33,10 +39,31 @@
         izz="${12.0 * 0.16 ** 2 / 2}"/>
     </inertial>
-    <visual>
-      <origin xyz="0 0 ${base_height / 2}" rpy="0 0 0"/>
-      <geometry>
-        <cylinder radius="0.16" length="${base_height}"/>
+    <visual name="mounting_foot">
+      <origin xyz="0 0 0.035" rpy="0 0 0"/>
+      <geometry>
+        <cylinder radius="0.225" length="0.07"/>
       </geometry>
       <material name="base_gray"/>
+    </visual>
+    <visual name="pedestal_shell">
+      <origin xyz="0 0 0.30" rpy="0 0 0"/>
+      <geometry>
+        <cylinder radius="0.14" length="0.48"/>
+      </geometry>
+      <material name="base_gray"/>
+    </visual>
+    <visual name="pedestal_trim">
+      <origin xyz="0 0 0.54" rpy="0 0 0"/>
+      <geometry>
+        <cylinder radius="0.165" length="0.035"/>
+      </geometry>
+      <material name="safety_yellow"/>
+    </visual>
+    <visual name="shoulder_support">
+      <origin xyz="0 0 0.62" rpy="0 0 0"/>
+      <geometry>
+        <cylinder radius="0.18" length="0.15"/>
+      </geometry>
+      <material name="rail_blue"/>
     </visual>
     <collision>
@@ -53,10 +80,24 @@
       <inertia ixx="0.0324" ixy="0" ixz="0" iyy="0.0324" iyz="0" izz="0.0600"/>
     </inertial>
-    <visual>
+    <visual name="yaw_housing">
       <origin xyz="0 0 0.04" rpy="0 0 0"/>
       <geometry>
-        <cylinder radius="0.20" length="0.08"/>
-      </geometry>
-      <material name="base_gray"/>
+        <cylinder radius="0.205" length="0.08"/>
+      </geometry>
+      <material name="rail_blue"/>
+    </visual>
+    <visual name="yaw_joint_band">
+      <origin xyz="0 0 0.012" rpy="0 0 0"/>
+      <geometry>
+        <cylinder radius="0.21" length="0.025"/>
+      </geometry>
+      <material name="tool_black"/>
+    </visual>
+    <visual name="yaw_cap">
+      <origin xyz="0 0 0.087" rpy="0 0 0"/>
+      <geometry>
+        <cylinder radius="0.17" length="0.025"/>
+      </geometry>
+      <material name="machined_steel"/>
     </visual>
     <collision>
@@ -79,10 +120,38 @@
         izz="0.1518625"/>
     </inertial>
-    <visual>
+    <visual name="radial_beam">
       <origin xyz="0.55 0 0" rpy="0 0 0"/>
       <geometry>
-        <box size="1.10 0.07 0.07"/>
+        <box size="1.10 0.13 0.11"/>
       </geometry>
       <material name="rail_blue"/>
+    </visual>
+    <visual name="guide_rail_left">
+      <origin xyz="0.55 0.055 0.064" rpy="0 0 0"/>
+      <geometry>
+        <box size="0.94 0.018 0.018"/>
+      </geometry>
+      <material name="machined_steel"/>
+    </visual>
+    <visual name="guide_rail_right">
+      <origin xyz="0.55 -0.055 0.064" rpy="0 0 0"/>
+      <geometry>
+        <box size="0.94 0.018 0.018"/>
+      </geometry>
+      <material name="machined_steel"/>
+    </visual>
+    <visual name="rail_end_stop_near">
+      <origin xyz="0.055 0 0" rpy="0 0 0"/>
+      <geometry>
+        <box size="0.07 0.16 0.14"/>
+      </geometry>
+      <material name="tool_black"/>
+    </visual>
+    <visual name="rail_end_stop_far">
+      <origin xyz="1.045 0 0" rpy="0 0 0"/>
+      <geometry>
+        <box size="0.07 0.16 0.14"/>
+      </geometry>
+      <material name="tool_black"/>
     </visual>
   </link>
@@ -92,9 +161,23 @@
       <inertia ixx="0.003333" ixy="0" ixz="0" iyy="0.003033" iyz="0" izz="0.003667"/>
     </inertial>
-    <visual>
-      <geometry>
-        <box size="0.14 0.16 0.12"/>
+    <visual name="saddle_housing">
+      <geometry>
+        <box size="0.23 0.24 0.12"/>
       </geometry>
       <material name="carriage_orange"/>
+    </visual>
+    <visual name="saddle_top_cover">
+      <origin xyz="0 0 0.072" rpy="0 0 0"/>
+      <geometry>
+        <box size="0.19 0.20 0.025"/>
+      </geometry>
+      <material name="tool_black"/>
+    </visual>
+    <visual name="vertical_axis_housing">
+      <origin xyz="0 0 -0.008" rpy="0 0 0"/>
+      <geometry>
+        <cylinder radius="0.105" length="0.085"/>
+      </geometry>
+      <material name="safety_yellow"/>
     </visual>
     <collision>
@@ -109,9 +192,23 @@
       <inertia ixx="0.002133" ixy="0" ixz="0" iyy="0.002133" iyz="0" izz="0.000683"/>
     </inertial>
-    <visual>
-      <geometry>
-        <box size="0.08 0.08 0.16"/>
-      </geometry>
-      <material name="base_gray"/>
+    <visual name="lift_actuator_shell">
+      <geometry>
+        <cylinder radius="0.075" length="0.17"/>
+      </geometry>
+      <material name="rail_blue"/>
+    </visual>
+    <visual name="lift_wiper_band">
+      <origin xyz="0 0 -0.09" rpy="0 0 0"/>
+      <geometry>
+        <cylinder radius="0.082" length="0.025"/>
+      </geometry>
+      <material name="tool_black"/>
+    </visual>
+    <visual name="exposed_lift_rod">
+      <origin xyz="0 0 -0.18" rpy="0 0 0"/>
+      <geometry>
+        <cylinder radius="0.032" length="0.19"/>
+      </geometry>
+      <material name="machined_steel"/>
     </visual>
     <collision>
@@ -126,9 +223,30 @@
       <inertia ixx="0.000209" ixy="0" ixz="0" iyy="0.000209" iyz="0" izz="0.000378"/>
     </inertial>
-    <visual>
-      <geometry>
-        <cylinder radius="0.055" length="0.03"/>
-      </geometry>
-      <material name="tool_black"/>
+    <visual name="suction_flange">
+      <geometry>
+        <cylinder radius="0.082" length="0.025"/>
+      </geometry>
+      <material name="tool_black"/>
+    </visual>
+    <visual name="tool_neck">
+      <origin xyz="0 0 0.048" rpy="0 0 0"/>
+      <geometry>
+        <cylinder radius="0.027" length="0.075"/>
+      </geometry>
+      <material name="machined_steel"/>
+    </visual>
+    <visual name="tool_actuator_cap">
+      <origin xyz="0 0 0.09" rpy="0 0 0"/>
+      <geometry>
+        <cylinder radius="0.052" length="0.035"/>
+      </geometry>
+      <material name="carriage_orange"/>
+    </visual>
+    <visual name="suction_lip">
+      <origin xyz="0 0 -0.018" rpy="0 0 0"/>
+      <geometry>
+        <cylinder radius="0.074" length="0.012"/>
+      </geometry>
+      <material name="safety_yellow"/>
     </visual>
     <collision>
